File: kicad/Kivipallur_left/Kivipallur_left.kicad_sch (KiCad schematic)
At the start: 21 parts, among them J1 TRRS, SW1 SW_Push, SW10 SW_Push, SW11 SW_Push, SW12 SW_Push, SW13 SW_Push, SW14 SW_Push, SW15 SW_Push, SW16 SW_Push, SW17 SW_Push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

Commit message: Add mounting holes to left hand schematic
Parts:
- added H1, H2, H3, H4, H5, H6, H7, H8: MountingHole, MountingHole:MountingHole_2.2mm_M2_Pad, symbol Mechanical:MountingHole

Commit message: Add left hand PCB design and gerbers
Connections:
- net INDEX_BOTTOM: now also U1.28 (P15); no longer U1.9 (P6)
- net INDEX_HOME: now also U1.11 (P8); no longer U1.8 (P5)
- net INDEX_TOP: now also U1.8 (P5); no longer U1.7 (P4)
- net INNER_BOTTOM: now also U1.27 (P14); no longer U1.6 (P3)
- net INNER_HOME: now also U1.10 (P7); no longer U1.5 (P2)
- net INNER_TOP: now also U1.9 (P6); no longer U1.31 (P10)
- net MIDDLE_BOTTOM: now also U1.29 (P16); no longer U1.12 (P9)
- net MIDDLE_HOME: now also U1.12 (P9); no longer U1.11 (P8)
- net MIDDLE_TOP: now also U1.7 (P4); no longer U1.10 (P7)
- net OUTER_TOP: now also U1.31 (P10); no longer U1.19 (P27)
- net PINKY_BOTTOM: now also U1.19 (P27); no longer U1.20 (P26)
- net PINKY_HOME: now also U1.26 (P13); no longer U1.29 (P16)
- net PINKY_TOP: now also U1.5 (P2); no longer U1.28 (P15)
- net RING_BOTTOM: now also U1.20 (P26); no longer U1.27 (P14)
- net RING_HOME: now also U1.25 (P12); no longer U1.26 (P13)
- net RING_TOP: now also U1.6 (P3); no longer U1.25 (P12)
Changed lines of the file:
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@@
 		)
 	)
-	(label "MIDDLE_TOP"
-		(at 25.4 99.06 0)
+	(label "PINKY_HOME"
+		(at 52.07 125.73 90)
+		(fields_autoplaced yes)
+		(effects
+			(font
+				(size 1.27 1.27)
+			)
+			(justify left bottom)
+		)
+	)
+	(label "INDEX_TOP"
+		(at 25.4 93.98 0)
 		(fields_autoplaced yes)
 		(effects
@@
 		)
 	)
-	(label "RING_TOP"
-		(at 49.53 125.73 90)
+	(label "INNER_TOP"
+		(at 25.4 96.52 0)
 		(fields_autoplaced yes)
 		(effects
@@
 		)
 	)
+	(label "OUTER_BOTTOM"
+		(at 83.82 88.9 180)
+		(fields_autoplaced yes)
+		(effects
+			(font
+				(size 1.27 1.27)
+			)
+			(justify right bottom)
+		)
+	)
 	(label "INDEX_TOP"
 		(at 133.35 26.67 0)
@@
 		)
 	)
+	(label "MIDDLE_HOME"
+		(at 25.4 104.14 0)
+		(fields_autoplaced yes)
+		(effects
+			(font
+				(size 1.27 1.27)
+			)
+			(justify left bottom)
+		)
+	)
 	(label "RING_HOME"
 		(at 74.93 39.37 0)
@@
 		)
 	)
-	(label "INDEX_HOME"
-		(at 25.4 93.98 0)
-		(fields_autoplaced yes)
-		(effects
-			(font
-				(size 1.27 1.27)
-			)
-			(justify left bottom)
-		)
-	)
 	(label "MIDDLE_TOP"
 		(at 104.14 26.67 0)
@@
 		)
 	)
-	(label "INNER_HOME"
-		(at 25.4 86.36 0)
+	(label "INNER_BOTTOM"
+		(at 54.61 125.73 90)
+		(fields_autoplaced yes)
+		(effects
+			(font
+				(size 1.27 1.27)
+			)
+			(justify left bottom)
+		)
+	)
+	(label "RING_BOTTOM"
+		(at 83.82 93.98 180)
+		(fields_autoplaced yes)
+		(effects
+			(font
+				(size 1.27 1.27)
+			)
+			(justify right bottom)
+		)
+	)
+	(label "RING_TOP"
+		(at 25.4 88.9 0)
+		(fields_autoplaced yes)
+		(effects
+			(font
+				(size 1.27 1.27)
+			)
+			(justify left bottom)
+		)
+	)
+	(label "MIDDLE_TOP"
+		(at 25.4 91.44 0)
 		(fields_autoplaced yes)
 		(effects
@@
 		)
 	)
-	(label "INNER_TOP"
-		(at 25.4 73.66 0)
-		(fields_autoplaced yes)
-		(effects
-			(font
-				(size 1.27 1.27)
-			)
-			(justify left bottom)
+	(label "PINKY_BOTTOM"
+		(at 83.82 91.44 180)
+		(fields_autoplaced yes)
+		(effects
+			(font
+				(size 1.27 1.27)
+			)
+			(justify right bottom)
 		)
 	)
@@
 		)
 	)
-	(label "INDEX_BOTTOM"
-		(at 25.4 96.52 0)
-		(fields_autoplaced yes)
-		(effects
-			(font
-				(size 1.27 1.27)
-			)
-			(justify left bottom)
-		)
-	)
 	(label "MIDDLE_HOME"
 		(at 104.14 39.37 0)
@@
 		)
 	)
-	(label "PINKY_BOTTOM"
-		(at 83.82 93.98 180)
-		(fields_autoplaced yes)
-		(effects
-			(font
-				(size 1.27 1.27)
-			)
-			(justify right bottom)
-		)
-	)
-	(label "INNER_BOTTOM"
-		(at 25.4 88.9 0)
-		(fields_autoplaced yes)
-		(effects
-			(font
-				(size 1.27 1.27)
-			)
-			(justify left bottom)
-		)
-	)
-	(label "PINKY_TOP"
-		(at 57.15 125.73 90)
-		(fields_autoplaced yes)
-		(effects
-			(font
-				(size 1.27 1.27)
-			)
-			(justify left bottom)
-		)
-	)
 	(label "THUMB_LEFT"
 		(at 133.35 64.77 0)
@@
 		)
 	)
+	(label "OUTER_TOP"
+		(at 25.4 73.66 0)
+		(fields_autoplaced yes)
+		(effects
+			(font
+				(size 1.27 1.27)
+			)
+			(justify left bottom)
+		)
+	)
 	(label "INDEX_HOME"
 		(at 133.35 39.37 0)
@@
 		)
 	)
-	(label "INDEX_TOP"
-		(at 25.4 91.44 0)
-		(fields_autoplaced yes)
-		(effects
-			(font
-				(size 1.27 1.27)
-			)
-			(justify left bottom)
-		)
-	)
 	(label "TRRS_RX"
 		(at 25.4 78.74 0)
@@
 		)
 	)
-	(label "RING_HOME"
-		(at 52.07 125.73 90)
-		(fields_autoplaced yes)
-		(effects
-			(font
-				(size 1.27 1.27)
-			)
-			(justify left bottom)
-		)
-	)
-	(label "OUTER_TOP"
-		(at 83.82 91.44 180)
-		(fields_autoplaced yes)
-		(effects
-			(font
-				(size 1.27 1.27)
-			)
-			(justify right bottom)
+	(label "PINKY_TOP"
+		(at 25.4 86.36 0)
+		(fields_autoplaced yes)
+		(effects
+			(font
+				(size 1.27 1.27)
+			)
+			(justify left bottom)
+		)
+	)
+	(label "INDEX_HOME"
+		(at 25.4 101.6 0)
+		(fields_autoplaced yes)
+		(effects
+			(font
+				(size 1.27 1.27)
+			)
+			(justify left bottom)
 		)
 	)
@@
 		)
 	)
-	(label "PINKY_HOME"
-		(at 59.69 125.73 90)
-		(fields_autoplaced yes)
-		(effects
-			(font
-				(size 1.27 1.27)
-			)
-			(justify left bottom)
-		)
-	)
 	(label "OUTER_TOP"
 		(at 16.51 26.67 0)
@@
 		)
 	)
-	(label "RING_BOTTOM"
-		(at 54.61 125.73 90)
-		(fields_autoplaced yes)
-		(effects
-			(font
-				(size 1.27 1.27)
-			)
-			(justify left bottom)
-		)
-	)
-	(label "OUTER_BOTTOM"
-		(at 83.82 88.9 180)
-		(fields_autoplaced yes)
-		(effects
-			(font
-				(size 1.27 1.27)
-			)
-			(justify right bottom)
+	(label "INDEX_BOTTOM"
+		(at 57.15 125.73 90)
+		(fields_autoplaced yes)
+		(effects
+			(font
+				(size 1.27 1.27)
+			)
+			(justify left bottom)
 		)
 	)
@@
 		)
 	)
+	(label "RING_HOME"
+		(at 49.53 125.73 90)
+		(fields_autoplaced yes)
+		(effects
+			(font
+				(size 1.27 1.27)
+			)
+			(justify left bottom)
+		)
+	)
 	(label "TRRS_TX"
 		(at 25.4 76.2 0)
@@
 		)
 	)
+	(label "MIDDLE_BOTTOM"
+		(at 59.69 125.73 90)
+		(fields_autoplaced yes)
+		(effects
+			(font
+				(size 1.27 1.27)
+			)
+			(justify left bottom)
+		)
+	)
 	(label "INNER_BOTTOM"
 		(at 162.56 52.07 0)
@@
 		)
 	)
-	(label "MIDDLE_HOME"
-		(at 25.4 101.6 0)
-		(fields_autoplaced yes)
-		(effects
-			(font
-				(size 1.27 1.27)
-			)
-			(justify left bottom)
-		)
-	)
-	(label "MIDDLE_BOTTOM"
-		(at 25.4 104.14 0)
-		(fields_autoplaced yes)
-		(effects
+	(label "INNER_HOME"
+		(at 25.4 99.06 0)
+		(fields_autoplaced yes)
+		(effects
