File: kicad/Kivipallur_left/Kivipallur_left.kicad_sch (KiCad schematic)
At the start: 29 parts, among them J1 TRRS, SW1 SW_Push, SW10 SW_Push, SW11 SW_Push, SW12 SW_Push, SW13 SW_Push, SW14 SW_Push, SW15 SW_Push, SW16 SW_Push, SW17 SW_Push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

Commit message: Add left hand PCB
Parts:
- U1: footprint PCM_marbastlib-xp-promicroish:Helios_AC -> PCM_marbastlib-xp-promicroish:Helios_ACH
Changed lines of the file:
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@@
 			)
 		)
-		(property "Footprint" "PCM_marbastlib-xp-promicroish:Helios_AC"
+		(property "Footprint" "PCM_marbastlib-xp-promicroish:Helios_ACH"
 			(at 54.61 114.3 0)
 			(effects
