File: kicad/Kivipallur_right/Kivipallur_right.kicad_pcb (KiCad board)
At the start: 2 copper layers, 158 x 105.1 mm, 30 parts, among them J1 TRRS, J2 Conn_01x07, SW1 SW_Push, SW10 SW_Push, SW11 SW_Push, SW12 SW_Push, SW13 SW_Push, SW14 SW_Push, SW15 SW_Push, SW16 SW_Push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

Commit message: Add finished right hand PCB
Routing:
- net /MOSI: track 37.2 -> 106.7 mm
- net /CS: track 29.8 -> 95.9 mm
- net +3V3: track 93.2 -> 158.8 mm, vias 0 -> 1
- net /SCK: track 51.9 -> 112.5 mm
- net /MISO: track 46.5 -> 105.1 mm, vias 1 -> 0
- net /THUMB_LEFT: track 119.9 -> 106.9 mm
- net /THUMB_RIGHT: track 103.3 -> 111.4 mm
- net /OUTER_TOP: track 158.3 -> 165.7 mm
- net /INNER_TOP: track 35.8 -> 40.6 mm
- net /OUTER_BOTTOM: track 197.8 -> 193.7 mm
- net /PINKY_BOTTOM: track 171.5 -> 167.6 mm
- net /RING_HOME: track 109.6 -> 112.4 mm
- net /TRRS_TX: track 5.95 -> 7.37 mm
- net /INNER_HOME: track 37.3 -> 38.5 mm
- net /INDEX_HOME: track 62.2 -> 61.2 mm
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- added copper zone on B.Cu, net GND
- added copper zone on F.Cu, net GND
